File: HEDGE2-OBC.kicad_sch (KiCad schematic)
At the start: 50 parts, among them J1 SMA-J-P-X-RA-TH1, U1 ADP7158ARDZ-3.3-R7, U3 SN74CBTLV3257PWR, U4 PCM5102AQPWRQ1, U5 TXS0102QDCURQ1

Commit message: Add PCM and SPI UART; begin layout update
Parts:
- removed U3: SN74CBTLV3257PWR, SN74CBTLV3257PWR:PW16, symbol SN74CBTLV3257PWR:SN74CBTLV3257PWR
- added C17, C18: 36p, Capacitor_SMD:C_0805_2012Metric, symbol Device:C_Small
- added IC1: SC16IS752IPW, SC16IS752IPW:SOP65P640X110-28N, symbol SC16IS752IPW:SC16IS752IPW
- added J2: 81_MMBX-S50-0-1/111_N, symbol SMA-J-P-X-RA-TH1:SMA-J-P-X-RA-TH1
- added R17, R18: 1k, Resistor_SMD:R_0805_2012Metric, symbol Device:R_Small_US
- added Y1: ABLS-LR-3.072MHZ-T, ABLS-LR-3.072MHZ-T:XTAL_ABLS-LR-3.072MHZ-T, symbol ABLS-LR-3.072MHZ-T:ABLS-LR-3.072MHZ-T
- renumbered C3 to C10, C4 to C11, C5 to C12, C17 to C13, C18 to C14, C19 to C15, C20 to C16, C13 to C19, C7 to C2, C14 to C20, C15 to C21, C16 to C22, C8 to C3, C9 to C4, C2 to C5, C10 to C6, C11 to C7, C12 to C8, C6 to C9, U4 to U2, U2 to U3, U5 to U4
Connections:
- net +3V3<CM4: now also R2.1, IC1.8 (VDD), R17.2
- net Associate/DIO5_XB: now also Module1.41 (GPIO25), IC1.19 (GPIO1/~{DTRB})
- net CAN_B_RXD: now also Module1.34 (GPIO5); no longer Module1.35 (ID_SC)
- net CAN_B_TXD: now also Module1.54 (GPIO4); no longer Module1.36 (ID_SD)
- net DIN/CONFIG/DIO14_XB: now also Module1.39 (GPIO8)
- net DOUT/DIO13_XB: now also Module1.40 (GPIO9)
- net DTR/SLEEP_RQ/DIO8_XB: now also Module1.45 (GPIO24)
- net GND: now also C17.1, C18.1, IC1.14 (SDA), IC1.22 (VSS), J2.2, J2.3, J2.4, J2.5, R18.2; no longer R2.1
- net GNSS_NRESET_IN: now also IC1.21 (GPIO3/~{RIB}); no longer Module1.48 (GPIO27)
- net GNSS_PPS: now also IC1.20 (GPIO2/~{CDB}); no longer Module1.46 (GPIO22)
- net GNSS_PV: now also IC1.18 (GPIO0/~{DSRB}); no longer Module1.50 (GPIO17)
- net GNSS_RXD2: now also IC1.3 (TXA); no longer Module1.34 (GPIO5)
- net GNSS_TXD2: now also IC1.4 (RXA); no longer Module1.54 (GPIO4)
- net ON_SLEEP/DIO9_XB: now also Module1.46 (GPIO22)
- net PTT_DMR: now also IC1.25 (GPIO4/~{DSRA}); no longer Module1.41 (GPIO25)
- net RESET_XB: now also Module1.48 (GPIO27)
- net T/R_DMR: now also IC1.26 (GPIO5/~{DTRA})
- net UART_RX_DMR: now also IC1.24 (RXB); no longer Module1.40 (GPIO9)
- net UART_TX_DMR: now also IC1.23 (TXB); no longer Module1.39 (GPIO8)
- net SPI3_RESET: now reaches Module1.29 (GPIO16)
- net SPI3_RESET: now also IC1.5 (~{RESET})
- net SPI3_SCLK: now reaches Module1.56 (GPIO3)
- net SPI3_SCLK: now also IC1.13 (SCL)
- net SPI3_MOSI: now reaches Module1.58 (GPIO2)
- net SPI3_MOSI: now also IC1.11 (A1)
- net AD0/DIO0_XB: no longer names the net of H2OBC1.15
- net AD1/DIO1/SPI_ATTN_XB: no longer names the net of H2OBC1.10
- net AD2/DIO2/SPI_CLK_XB: no longer names the net of H2OBC1.06
- net AD3/DIO3/SPI_SSEL_XB: no longer names the net of H2OBC1.05
- net Antenna: no longer names the net of J1.1, U3.21 (ANT)
- net Antenna: now also J2.1
- net CS_DMR: no longer names the net of H2OBC1.24
- net CTS/DIO7_XB: no longer names the net of H2OBC1.04
- net DIO10/PWM0_XB: no longer names the net of H2OBC1.12
- net DIO11/PWM1_XB: no longer names the net of H2OBC1.14
- net DIO12/SPI_MISO_XB: no longer names the net of H2OBC1.08
- net DIO4/SPI_MOSI_XB: no longer names the net of H2OBC1.07
- net HST_RXD_DMR: no longer names the net of H2OBC1.25
- net HST_TXD_DMR: no longer names the net of H2OBC1.27
- net I2C_EN: no longer names the net of R2.2, U4.6 (OE)
- net I2C_EN: no longer Module1.30 (GPIO6)
- net LINE_OUT_DMR: no longer names the net of H2OBC1.20
- net NDTR_XB: no longer names the net of H2OBC1.17
- net RTS/DIO6_XB: no longer names the net of H2OBC1.03
- net SPKEN_DMR: no longer names the net of H2OBC1.23
- new net: C18.2, IC1.7 (XTAL2), Y1.2
- new net: IC1.9 (I2C), R18.1
- new net: C17.2, IC1.6 (XTAL1), Y1.1
- new net SPI3_CE0_0: IC1.10 (A0), Module1.36 (ID_SD)
- new net SPI3_INT: IC1.15 (~{IRQ}), R17.1
- new net SPI3_MISO: IC1.12 (SO), Module1.35 (ID_SC)
- no-connect marks 179 -> 199
Other:
- note added: "CM4 SERIAL INTERFACE ASSIGNMENTS"
- note added: "LINE_OUT_DMR (unused)"
- note removed: "GNSS"
- note removed: "Housekeeping (TEMP)"
- note removed: "Housekeeping (VOLT/CURR)"
- note removed: "I2C0 BUS"
- note removed: "RS-485"
- note removed: "SPACECRAFT BUS"
- note removed: "SpaceCAN (CANbus)"
- moved on the sheet: C1, C10, C11, C12, C13, C14, C15, C16, C2, C3, C4, C5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

Commit message: Continue layout update
Parts:
- removed C17, C18: 36p, Capacitor_SMD:C_0805_2012Metric, symbol Device:C_Small
- removed Y1: ABLS-LR-3.072MHZ-T, ABLS-LR-3.072MHZ-T:XTAL_ABLS-LR-3.072MHZ-T, symbol ABLS-LR-3.072MHZ-T:ABLS-LR-3.072MHZ-T
- added C21: 10p, Capacitor_SMD:C_0805_2012Metric, symbol Device:C_Small
- added X1: XLH536003.072000I, XLH53xxxxxx:SON6_XLH5_5p0x3p2-1p27_REN_REN, symbol XLH53xxxxxx:XLH535100.000000X
- renumbered C19 to C17, C20 to C18, C21 to C19, C22 to C20, R18 to R11, R17 to R12, R11 to R13, R12 to R14
Connections:
- net +3V3<CM4: now also C21.2, X1.6 (VDD)
- net Associate/DIO5_XB: no longer Module1.41 (GPIO25)
- net GND: now also C21.1, X1.3 (GND)
- net at IC1.6 (XTAL1): now also X1.4 (OUT)
- no-connect marks 199 -> 203
Other:
- moved on the sheet: C13, C14, C15, C16, C2, C3, C4, C6, C7, C8, C9, IC1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

Commit message: Add IMU; eliminate environmental sensor; finish layout
Parts:
- added C17: 1u, Capacitor_SMD:C_0805_2012Metric, symbol Device:C_Small
- added C22, C23: 100n, Capacitor_SMD:C_0805_2012Metric, symbol Device:C_Small
- added R2, R3: 10k, Resistor_SMD:R_0805_2012Metric, symbol Device:R_Small_US
- added U4: BNO055, BNO055:LGA28R50P4X10_380X520X100, symbol BNO055:BNO055
- added Y1: QT325S-32.768MAHE-T, Crystal:Crystal_SMD_3225-4Pin_3.2x2.5mm, symbol Device:Crystal_GND24
- renumbered C17 to C18, C18 to C19, C19 to C20, C20 to C21, C21 to C24, R8 to R10, R9 to R11, R10 to R12, R11 to R13, R12 to R14, R13 to R15, R14 to R16, R2 to R4, R3 to R5, R4 to R6, R5 to R7, R6 to R8, R7 to R9, U4 to U5
Connections:
- net +3V3<CM4: now also C22.1, C23.1, R2.2, R3.2, U4.28 (VDDIO), U4.3 (VDD)
- net GND: now also C17.2, C22.2, C23.2, U4.17 (COM3), U4.18 (COM2), U4.2 (GND), U4.25 (GNDIO), U4.5 (PS1), U4.6 (PS0), Y1.2 (G), Y1.4 (G)
- net SCL0_3V3: now also U4.19 (COM1)
- net SDA0_3V3: now also U4.20 (COM0)
- net INT_BNO: now reaches Module1.30 (GPIO6)
- net INT_BNO: now also U4.14 (INT)
- net NRESET_BNO: now reaches Module1.44 (GPIO10)
- net NRESET_BNO: now also R2.1, U4.11 (NRESET)
- removed net BATT: H2OBC1.41, H2OBC1.42, H2OBC1.43, H2OBC1.44, H2OBC1.45, H2OBC1.46
- net ENA_PWR_5: no longer names the net of H2OBC1.33
- net ENA_PWR_6: no longer names the net of H2OBC1.35
- net ENA_PWR_7: no longer names the net of H2OBC1.37
- net ENA_PWR_8: no longer names the net of H2OBC1.39
- net PWR_5: no longer names the net of H2OBC1.34
- net PWR_6: no longer names the net of H2OBC1.36
- net PWR_7: no longer names the net of H2OBC1.38
- net PWR_8: no longer names the net of H2OBC1.40
- net UART_E_RX renamed UART_SCI_RX
- net UART_E_TX renamed UART_SCI_TX
- new net: R3.1, U4.4 (NBOOT_LOAD_PIN)
- new net: C17.1, U4.9 (CAP)
- new net XIN32: U4.27 (XIN32), Y1.1
- new net XOUT32: U4.26 (XOUT32), Y1.3
- no-connect marks 203 -> 210
Other:
- removed sheet MAX6635_GNSS
- note added: "0x28"
- note removed: "0x48"
