File: HEDGE2-OBC.kicad_sch (KiCad schematic)
At the start: 62 parts, among them IC1 SC16IS752IPW, J1 SMA-J-P-X-RA-TH1, J2 81_MMBX-S50-0-1/111_N, U1 ADP7158ARDZ-3.3-R7, U2 PCM5102AQPWRQ1, U4 BNO055, U5 TXS0102QDCURQ1, X1 XLH536003.072000I, Y1 QT325S-32.768MAHE-T

Commit message: Final cleanup
Parts:
- C10: DigiKey Part Number (none) -> 490-GRM21BZ71E106KE15KCT-ND
- C13, C16: DigiKey Part Number (none) -> 718-TP8R106M016CCT-ND
- C14: renamed from C15; DigiKey Part Number (none) -> 720-GA0805Y104JXABT31GCT-ND
- C15: renamed from C14; DigiKey Part Number (none) -> 720-GA0805Y104JXABT31GCT-ND
- C17: DigiKey Part Number (none) -> 1276-1029-1-ND
- C2: DigiKey Part Number (none) -> 445-174216-1-ND
- C22, C23: DigiKey Part Number (none) -> 478-KAM21BR71H104KTCT-ND
- C24: DigiKey Part Number (none) -> 478-06035C100K4T4ACT-ND
- C3: renamed from C9; DigiKey Part Number (none) -> 1276-6555-1-ND
- C4: renamed from C3; DigiKey Part Number (none) -> 718-TP8R106M016CCT-ND
- C5: renamed from C4; DigiKey Part Number (none) -> 718-TP8R106M016CCT-ND
- C6: renamed from C5; DigiKey Part Number (none) -> 490-GRM21BZ71E106KE15KCT-ND
- C7: renamed from C6; DigiKey Part Number (none) -> 445-174216-1-ND
- C8: renamed from C7; DigiKey Part Number (none) -> 720-GA0805Y104JXABT31GCT-ND
- C9: renamed from C8; DigiKey Part Number (none) -> 720-GA0805Y104JXABT31GCT-ND
- JP1: value OEM719B ENABLE -> GNSS EN
- JP2: value CM4 ENABLE -> CM4 EN
- JP3: value LDO 3V3 ENABLE -> 3V3 EN
- R1: DigiKey Part Number (none) -> 738-RMCA0805FT470R-HPCT-ND
- R2, R3: DigiKey Part Number (none) -> RNCP0805FTD10K0CT-ND
- R4: DigiKey Part Number 541-10.0KCCT-ND -> RNCP0805FTD10K0CT-ND
- X1: DigiKey Part Number (none) -> 631-1272-ND
- Y1: DigiKey Part Number (none) -> 4981-QT325S-32.768MAHE-TCT-ND
Other:
- note removed: "LINE_OUT_DMR (unused)"
- moved on the sheet: C14, C16, C3, R1
